Commit message: added humble support
this now uses gazebo ignition and tugbot_warehouse.sdf as world

File: description/depth_camera.xacro (robot description, xacro)
@@ -21,13 +21,24 @@
     <link name="camera_link_optical"></link>
     <gazebo reference="camera_link">
-        <material>Gazebo/Red</material>
-        <sensor name="camera" type="depth">
+        <visual>
+            <material>
+                <ambient>1 0 0 1</ambient>
+                <diffuse>1 0 0 1</diffuse>
+                <specular>1 0 0 1</specular>
+            </material>
+        </visual>
+        <!-- CHANGED: Type is now rgbd_camera (Color + Depth + Points) -->
+        <sensor name="camera" type="rgbd_camera">
             <pose> 0 0 0 0 0 0 </pose>
             <visualize>true</visualize>
             <update_rate>10</update_rate>
+            <!-- CHANGED: Base topic is just "camera" -->
+            <!-- Ign generates: /camera/image, /camera/depth_image, /camera/points -->
+            <topic>camera</topic>
+            <gz_frame_id>camera_link</gz_frame_id>
             <camera>
                 <horizontal_fov>1.089</horizontal_fov>
                 <image>
-                    <format>B8G8R8</format>
+                    <format>R8G8B8</format>
                     <width>640</width>
                     <height>480</height>
@@ -38,9 +49,4 @@
                 </clip>
             </camera>
-            <plugin name="camera_controller" filename="libgazebo_ros_camera.so">
-                <frame_name>camera_link_optical</frame_name>
-                <min_depth>0.1</min_depth>
-                <max_depth>100.0</max_depth>
-            </plugin>
         </sensor>
     </gazebo>

File: description/gazebo_control.xacro (robot description, xacro)
@@ -2,19 +2,24 @@
 <robot xmlns:xacro="http://www.ros.org/wiki/xacro">
     <gazebo>
-        <plugin name='diff_drive' filename='libgazebo_ros_diff_drive.so'>
+        <!-- Ignition Gazebo Diff Drive Plugin -->
+        <plugin filename="ignition-gazebo-diff-drive-system" name="ignition::gazebo::systems::DiffDrive">
             <!-- Wheel Information -->
             <left_joint>left_wheel_joint</left_joint>
             <right_joint>right_wheel_joint</right_joint>
             <wheel_separation>0.35</wheel_separation>
-            <wheel_diameter>0.1</wheel_diameter>
+            <wheel_radius>0.05</wheel_radius>
             <!-- Limits -->
-            <max_wheel_torque>200</max_wheel_torque>
-            <max_wheel_acceleration>10.0</max_wheel_acceleration>
-            <!-- Output -->
-            <odometry_frame>odom</odometry_frame>
-            <robot_base_frame>base_link</robot_base_frame>
-            <publish_odom>true</publish_odom>
-            <publish_odom_tf>true</publish_odom_tf>
-            <publish_wheel_tf>false</publish_wheel_tf>
+            <max_linear_acceleration>10</max_linear_acceleration>
+            <!-- Input / Output -->
+            <topic>cmd_vel</topic> <!-- Ignition Topic -->
+            <odom_topic>odom</odom_topic> <!-- Ignition Topic -->
+            <tf_topic>tf</tf_topic>
+            <frame_id>odom</frame_id>
+            <child_frame_id>base_link</child_frame_id>
+            <odom_publish_frequency>30</odom_publish_frequency>
+        </plugin>
+        <!-- Helper plugin to publish Joint States (Optional but good for Rviz) -->
+        <plugin filename="ignition-gazebo-joint-state-publisher-system" name="ignition::gazebo::systems::JointStatePublisher">
+            <topic>joint_states</topic>
         </plugin>
     </gazebo>

File: description/lidar.xacro (robot description, xacro)
@@ -21,13 +21,25 @@
     </link>
     <gazebo reference="laser_frame">
-        <material>Gazebo/Red</material>
-        <sensor name="laser" type="ray">
+        <visual>
+            <material>
+                <ambient>1 0 0 1</ambient>
+                <diffuse>1 0 0 1</diffuse>
+                <specular>1 0 0 1</specular>
+            </material>
+        </visual>
+        <!-- IGNITION SENSOR SETUP -->
+        <sensor name="laser" type="gpu_lidar">
             <pose> 0 0 0 0 0 0 </pose>
             <visualize>true</visualize>
             <update_rate>10</update_rate>
+            <!-- This tag sets the Ignition topic name -->
+            <topic>scan</topic>
+            <!-- This tag sets the frame ID for the ROS message -->
+            <gz_frame_id>laser_frame</gz_frame_id>
             <ray>
                 <scan>
                     <horizontal>
                         <samples>360</samples>
+                        <resolution>1</resolution>
                         <min_angle>-3.14</min_angle>
                         <max_angle>3.14</max_angle>
@@ -39,11 +51,4 @@
                 </range>
             </ray>
-            <plugin name="laser_controller" filename="libgazebo_ros_ray_sensor.so">
-                <ros>
-                    <argument>out:=scan</argument>
-                </ros>
-                <output_type>sensor_msgs/LaserScan</output_type>
-                <frame_name>laser_frame</frame_name>
-            </plugin>
         </sensor>
     </gazebo>

File: description/robot_core.xacro (robot description, xacro)
@@ -6,5 +6,8 @@
     <material name="blue"><color rgba="0.2 0.2 1 1"/></material>
     <material name="black"><color rgba="0 0 0 1"/></material>
+    <material name="red"><color rgba="1 0 0 1"/></material>
+    <!-- BASE LINK -->
     <link name="base_link"/>
+    <!-- CHASSIS -->
     <joint name="chassis_joint" type="fixed">
         <parent link="base_link"/>
@@ -29,6 +32,13 @@
     </link>
     <gazebo reference="chassis">
-        <material>Gazebo/White</material>
+        <visual>
+            <material>
+                <ambient>1 1 1 1</ambient>
+                <diffuse>1 1 1 1</diffuse>
+                <specular>1 1 1 1</specular>
+            </material>
+        </visual>
     </gazebo>
+    <!-- LEFT WHEEL -->
     <joint name="left_wheel_joint" type="continuous">
         <parent link="base_link"/>
@@ -52,6 +62,13 @@
     </link>
     <gazebo reference="left_wheel">
-        <material>Gazebo/Blue</material>
+        <visual>
+            <material>
+                <ambient>0.2 0.2 1 1</ambient>
+                <diffuse>0.2 0.2 1 1</diffuse>
+                <specular>0.2 0.2 1 1</specular>
+            </material>
+        </visual>
     </gazebo>
+    <!-- RIGHT WHEEL -->
     <joint name="right_wheel_joint" type="continuous">
         <parent link="base_link"/>
@@ -75,6 +92,13 @@
     </link>
     <gazebo reference="right_wheel">
-        <material>Gazebo/Blue</material>
+        <visual>
+            <material>
+                <ambient>0.2 0.2 1 1</ambient>
+                <diffuse>0.2 0.2 1 1</diffuse>
+                <specular>0.2 0.2 1 1</specular>
+            </material>
+        </visual>
     </gazebo>
+    <!-- CASTER WHEEL -->
     <joint name="caster_wheel_joint" type="fixed">
         <parent link="chassis"/>
@@ -97,7 +121,22 @@
     </link>
     <gazebo reference="caster_wheel">
-        <material>Gazebo/Black</material>
-        <mu1 value="0.001"/>
-        <mu2 value="0.001"/>
+        <visual>
+            <material>
+                <ambient>0 0 0 1</ambient>
+                <diffuse>0 0 0 1</diffuse>
+                <specular>0 0 0 1</specular>
+            </material>
+        </visual>
+        <!-- Friction for Ignition/Gazebo Fortress -->
+        <collision>
+            <surface>
+                <friction>
+                    <ode>
+                        <mu>0.001</mu>
+                        <mu2>0.001</mu2>
+                    </ode>
+                </friction>
+            </surface>
+        </collision>
     </gazebo>
 </robot>
