Commit message: added slam toolbox

File: description/lidar.xacro (robot description, xacro)
@@ -47,4 +47,5 @@
                 </range>
             </ray>
+            <topic>scan</topic>
         </sensor>
     </gazebo>

File: description/robot_core.xacro (robot description, xacro)
@@ -1,5 +1,6 @@
 <?xml version="1.0"?>
-<robot xmlns:xacro="http://www.ros.org/wiki/xacro">
+<robot xmlns:xacro="http://www.ros.org/wiki/xacro" name="mybot">
     <xacro:include filename="inertial_macros.xacro" />
+    <!-- MATERIALS -->
     <material name="white"><color rgba="1 1 1 1"/></material>
     <material name="orange"><color rgba="1 0.3 0.1 1"/></material>
@@ -9,5 +10,5 @@
     <!-- BASE LINK -->
     <link name="base_link"/>
-    <!-- CHASSIS -->
+    <!-- CHASSIS LINK -->
     <joint name="chassis_joint" type="fixed">
         <parent link="base_link"/>
@@ -69,4 +70,17 @@
             </material>
         </visual>
+        <!-- ADDED FRICTION FOR LEFT WHEEL -->
+        <collision>
+            <surface>
+                <friction>
+                    <ode>
+                        <mu>1.0</mu>        <!-- High friction for driving -->
+                        <mu2>1.0</mu2>      <!-- High friction for driving -->
+                        <slip1>0.0</slip1> <!-- Small amount of slip for realism -->
+                        <slip2>0.0</slip2>
+                    </ode>
+                </friction>
+            </surface>
+        </collision>
     </gazebo>
     <!-- RIGHT WHEEL -->
@@ -99,4 +113,17 @@
             </material>
         </visual>
+        <!-- ADDED FRICTION FOR RIGHT WHEEL -->
+        <collision>
+            <surface>
+                <friction>
+                    <ode>
+                        <mu>1.0</mu>        <!-- High friction for driving -->
+                        <mu2>1.0</mu2>      <!-- High friction for driving -->
+                        <slip1>0.0</slip1> <!-- Small amount of slip for realism -->
+                        <slip2>0.0</slip2>
+                    </ode>
+                </friction>
+            </surface>
+        </collision>
     </gazebo>
     <!-- CASTER WHEEL -->
@@ -132,6 +159,6 @@
                 <friction>
                     <ode>
-                        <mu>0.001</mu>
-                        <mu2>0.001</mu2>
+                        <mu>0.01</mu>
+                        <mu2>0.01</mu2>
                     </ode>
                 </friction>
@@ -139,3 +166,35 @@
         </collision>
     </gazebo>
+    <gazebo>
+        <!-- Diff Drive Plugin -->
+        <plugin filename="libignition-gazebo-diff-drive-system.so" name="ignition::gazebo::systems::DiffDrive">
+            <left_joint>left_wheel_joint</left_joint>
+            <right_joint>right_wheel_joint</right_joint>
+            <!-- Kinematics based on your link geometry -->
+            <wheel_separation>0.35</wheel_separation>
+            <wheel_radius>0.05</wheel_radius>
+            <!-- Limits -->
+            <max_linear_acceleration>1</max_linear_acceleration>
+            <min_linear_acceleration>-1</min_linear_acceleration>
+            <max_angular_acceleration>2</max_angular_acceleration>
+            <min_angular_acceleration>-2</min_angular_acceleration>
+            <max_linear_velocity>0.5</max_linear_velocity>
+            <min_linear_velocity>-0.5</min_linear_velocity>
+            <max_angular_velocity>1</max_angular_velocity>
+            <min_angular_velocity>-1</min_angular_velocity>
+            <!-- Output Topics -->
+            <topic>cmd_vel</topic>
+            <odom_topic>odom</odom_topic>
+            <tf_topic>tf</tf_topic>
+            <frame_id>odom</frame_id>
+            <child_frame_id>base_link</child_frame_id>
+            <odom_publisher_frequency>30</odom_publisher_frequency>
+        </plugin>
+        <!-- Joint State Publisher (Publishes TFs for wheels) -->
+        <plugin filename="libignition-gazebo-joint-state-publisher-system.so" name="ignition::gazebo::systems::JointStatePublisher">
+            <topic>joint_states</topic>
+            <joint_name>left_wheel_joint</joint_name>
+            <joint_name>right_wheel_joint</joint_name>
+        </plugin>
+    </gazebo>
 </robot>
